File: kicad/Mains_monitor.kicad_sch (KiCad schematic)
At the start: 1 part, among them U1 ESP32-WROOM-32

Commit message: Design power supply circuit
Parts:
- removed U1: ESP32-WROOM-32, RF_Module:ESP32-WROOM-32, symbol RF_Module:ESP32-WROOM-32
- added U1: ESP32-C3-WROOM-02, RF_Module:ESP32-C3-WROOM-02, symbol RF_Module:ESP32-C3-WROOM-02
Connections:
- new net +3V3: U1.1 (3V3)
- new net GND: U1.19 (GND), U1.9 (GND)
Other:
- removed sheet non_isolated_supply.sch
- sheet energy monitor ports: added TX; removed none
