File: kicad/current_sense_ckt.kicad_sch (KiCad schematic)
At the start: 6 parts, among them T1 CST2010

Commit message: Add rev0 schematic
Parts:
- removed C3, C6: 33n, symbol Device:C
- removed R3: 1, symbol Device:R
- removed R6, R7: 1k, symbol Device:R
- removed T1: CST2010, Transformer_SMD:Transformer_Coilcraft_CST2010, symbol Transformer:CST2010
