File: kicad/energy_monitor.kicad_sch (KiCad schematic)
At the start: 5 parts

Commit message: Design power supply circuit
Parts:
- removed R10, R11, R12, R13, R9: 470k, symbol Device:R
- added C4: 100n, symbol Device:C_Polarized_US
- added C5: 1u, symbol Device:C_Polarized_US
- added U3: HLW8032, Package_SO:SSOP-8_3.9x5.05mm_P1.27mm, symbol mains_mon:HLW8032
Connections:
- new net +5V: C4.1, C5.1, U3.1 (VDD)
- new net GND: C4.2, C5.2, U3.5 (GND)
- new net IN: U3.3 (IN)
- new net IP: U3.2 (IP)
- new net VP: U3.4 (VP)
- no-connect marks 0 -> 2

Commit message: Add rev0 schematic
Parts:
- removed C4: 100n, symbol Device:C_Polarized_US
- removed C5: 1u, symbol Device:C_Polarized_US
- added C10: 100n, Capacitor_SMD:C_0805_2012Metric_Pad1.18x1.45mm_HandSolder, symbol Device:C
- added C9: 10u, Capacitor_SMD:C_0805_2012Metric_Pad1.18x1.45mm_HandSolder, symbol Device:C
- added Q2: BS170, Package_TO_SOT_THT:TO-92_Inline, symbol Transistor_FET:BS170
- added R10, R9: 10k, symbol Device:R
Connections:
- net +5V: now also C10.1, C9.1, R10.1
- net GND: now also C10.2, C9.2
- net at U3.6 (TX): now also Q2.1 (D), R10.2
- new net +3V3: Q2.2 (G), R9.1
- new net MCU_RX: Q2.3 (S), R9.2
Other:
- note added: "Level Shifter for 5v to 3v3"
- title: Isolated Supply -> Energy Monitor
- moved on the sheet: U3
