File: kicad/isolated supply.kicad_sch (KiCad schematic)
At the start: 4 parts

Commit message: Design power supply circuit
Parts:
- removed PS1: HLK-2M03, Converter_ACDC:Converter_ACDC_Hi-Link_HLK-2Mxx, symbol Converter_ACDC:HLK-2M03
- added PS1: HLK-5M05, Converter_ACDC:Converter_ACDC_Hi-Link_HLK-5Mxx, symbol Converter_ACDC:HLK-5M05
- added U2: AMS1117-3.3, Package_TO_SOT_SMD:SOT-223-3_TabPin2, symbol Regulator_Linear:AMS1117-3.3
Connections:
- net +3V3: now also U2.2 (VO); no longer C?.1, L?.2
- net ACOUT_1: now also PS1.1 (AC/L)
- net ACOUT_2: now also PS1.2 (AC/N)
- net at C?.1, L?.1: now also PS1.4 (+Vout)
- net GND2 renamed GND
- net GND: now also PS1.3 (-Vout), U2.1 (GND)
- new net +5V: C?.1, L?.2, U2.3 (VI)
Other:
- moved on the sheet: C?, L?

Commit message: Add rev0 schematic
Parts:
- removed C? (x2): 470u, symbol Device:C
- removed L?: 22u, symbol Device:L
- removed PS1: HLK-5M05, Converter_ACDC:Converter_ACDC_Hi-Link_HLK-5Mxx, symbol Converter_ACDC:HLK-5M05
- removed U2: AMS1117-3.3, Package_TO_SOT_SMD:SOT-223-3_TabPin2, symbol Regulator_Linear:AMS1117-3.3
