File: kicad/mains input.kicad_sch (KiCad schematic)
At the start: 12 parts, among them J1 120VAC, J2 LOAD, T1 CST2010

Commit message: Design power supply circuit
Parts:
- removed FL2: Choke_Schaffner_RN102-0.3-02-12M, Inductor_THT:Choke_Schaffner_RN102-04-14.0x14.0mm, symbol Filter:Choke_Schaffner_RN102-0.3-02-12M
- removed R1: 100, symbol Device:R
- removed R2, R3: 12k, symbol Device:R
- removed T1: CST2010, Transformer_SMD:Transformer_Coilcraft_CST2010, symbol Transformer:CST2010
- F1: value 500mA -> 1.5A
Connections:
- net Current Sense Ckt/Load_N: now reaches J2.1 (Pin_1)
- net Switching Ckt/Load_L renamed Current Sense Ckt/Load_L
- net VP renamed Switching Ckt/AC_L
Other:
- added sheet Current Sense Ckt (current_sense_ckt.kicad_sch)
- added sheet Voltage Sense Ckt (voltage_sense_ckt.kicad_sch)

Commit message: Add rev0 schematic
Parts:
- added A1: Adafruit_Feather_HUZZAH32_ESP32, Module:Adafruit_Feather, symbol MCU_Module:Adafruit_Feather_HUZZAH32_ESP32
- added C2: 10u, Capacitor_SMD:C_0805_2012Metric_Pad1.18x1.45mm_HandSolder, symbol Device:C
- added C3, C4, C5: 33n, Capacitor_SMD:C_0805_2012Metric_Pad1.18x1.45mm_HandSolder, symbol Device:C
- added C6: 100n, Capacitor_SMD:C_0805_2012Metric_Pad1.18x1.45mm_HandSolder, symbol Device:C
- added D1: D, symbol Device:D
- added FL3: choke, Inductor_THT:Choke_Schaffner_RN102-04-14.0x14.0mm, symbol Filter:Choke_Schaffner_RN102-0.3-02-12M
- added K2: SANYOU_SRD_Form_C, Relay_THT:Relay_SPDT_SANYOU_SRD_Series_Form_C, symbol Relay:SANYOU_SRD_Form_C
- added PS1: HLK-5M05, Converter_ACDC:Converter_ACDC_Hi-Link_HLK-5Mxx, symbol Converter_ACDC:HLK-5M05
- added Q3: NPN, symbol Simulation_SPICE:NPN
- added Q4: BS170, Package_TO_SOT_THT:TO-92_Inline, symbol Transistor_FET:BS170
- added R1, R2: 10k, symbol Device:R
- added R11: 3.3k, symbol Device:R
- added R12, R13: 12k, symbol Device:R
- added R14: 49.9, symbol Device:R
- added R15, R6, R7: 1k, symbol Device:R
- added R3: 1, symbol Device:R
- added T1: CST2010, Transformer_SMD:Transformer_Coilcraft_CST2010, symbol Transformer:CST2010
- added U1: HLW8032, Package_SO:SSOP-8_3.9x5.05mm_P1.27mm, symbol mains_mon:HLW8032
- C1: footprint (none) -> Capacitor_THT:C_Rect_L18.0mm_W5.0mm_P15.00mm_FKS3_FKP3
Connections:
- net AC_N: now reaches C1.2, FL1.3, J1.N (Pin_1), RV1.2
- net AC_N: now also R13.2
- net ACOUT-1: no longer names the net of FL1.2
- net ACOUT-1: now also PS1.1 (AC/L)
- net ACOUT-2: no longer names the net of FL1.4
- net ACOUT-2: now also PS1.2 (AC/N)
- net Current Sense Ckt/Load_L renamed LOAD_L
- net LOAD_L: now also T1.11
- net Current Sense Ckt/Load_N renamed LOAD_N
- net Switching Ckt/AC_L renamed AC_L
- net AC_L: now also R12.1, T1.12
- new net: FL3.4, R14.2, R15.1
- new net: D1.2 (A), K2.2, Q3.1 (C)
- new net: Q3.2 (B), R11.2
- new net: FL3.1, R13.1
- new net: FL3.2, R12.2
- new net: R3.1, R6.1, T1.4
- new net +3V3: Q4.2 (G), R2.1
- new net +5V: C2.2, C6.1, D1.1 (K), K2.5, PS1.4 (+Vout), R1.1, U1.1 (VDD)
- new net E_TX: Q4.1 (D), R1.2, U1.6 (TX)
- new net GND: A1.4 (GND), C2.1, C3.2, C4.1, C5.2, C6.2, FL3.3, PS1.3 (-Vout), Q3.3 (E), R14.1, R3.2, R7.1, T1.2, U1.5 (GND)
- new net IN: C4.2, R7.2, U1.3 (IN)
- new net IO14: A1.19 (A6/IO14), R11.1
- new net IP: C3.1, R6.2, U1.2 (IP)
- new net MCU_RX: A1.14 (RX/IO16), Q4.3 (S), R2.2
- new net VP: C5.1, R15.2, U1.4 (VP)
- no-connect marks 0 -> 27
Other:
- removed sheet Current Sense Ckt
- removed sheet Switching Ckt
- removed sheet Voltage Sense Ckt
- note added: "Current Sense Transformer"
- note added: "Current type voltage transformer"
- note added: "Level Shifter for 5v to 3v3"
- moved on the sheet: C1, F1, FL1, J1, J2, RV1, TH1
